Commit message: Correct joint origin but the orientation is 90 deg offset

File: robotic_description/urdf/robotic.xacro (robot description, xacro)
@@ -84,12 +84,72 @@
   </collision>
 </link>
+<link name="WRIST_1">
+  <inertial>
+    <origin xyz="-6.006126105094087e-06 0.022392627588266822 -0.0001885326507429853" rpy="0 0 0"/>
+    <mass value="0.062244194694843255"/>
+    <inertia ixx="2.4e-05" iyy="2.1e-05" izz="1.8e-05" ixy="-0.0" iyz="-0.0" ixz="0.0"/>
+  </inertial>
+  <visual>
+    <origin xyz="-0.0 -0.407987 -0.0001" rpy="0 0 0"/>
+    <geometry>
+      <mesh filename="file://$(find robotic_description)/meshes/WRIST_1.stl" scale="0.001 0.001 0.001"/>
+    </geometry>
+    <material name="silver"/>
+  </visual>
+  <collision>
+    <origin xyz="-0.0 -0.407987 -0.0001" rpy="0 0 0"/>
+    <geometry>
+      <mesh filename="file://$(find robotic_description)/meshes/WRIST_1.stl" scale="0.001 0.001 0.001"/>
+    </geometry>
+  </collision>
+</link>
+<link name="finger_1_1">
+  <inertial>
+    <origin xyz="-0.0007126631883796379 0.016327909388517248 0.05456077201686822" rpy="0 0 0"/>
+    <mass value="0.0544277408008124"/>
+    <inertia ixx="1.4e-05" iyy="8e-06" izz="1.4e-05" ixy="3e-06" iyz="-3e-06" ixz="1e-06"/>
+  </inertial>
+  <visual>
+    <origin xyz="-0.006 -0.447874 0.0298" rpy="0 0 0"/>
+    <geometry>
+      <mesh filename="file://$(find robotic_description)/meshes/finger_1_1.stl" scale="0.001 0.001 0.001"/>
+    </geometry>
+    <material name="silver"/>
+  </visual>
+  <collision>
+    <origin xyz="-0.006 -0.447874 0.0298" rpy="0 0 0"/>
+    <geometry>
+      <mesh filename="file://$(find robotic_description)/meshes/finger_1_1.stl" scale="0.001 0.001 0.001"/>
+    </geometry>
+  </collision>
+</link>
+<link name="finger_1_2">
+  <inertial>
+    <origin xyz="0.0007126631883832904 0.016327909388515915 0.0002391557905749818" rpy="0 0 0"/>
+    <mass value="0.0544277408008124"/>
+    <inertia ixx="1.4e-05" iyy="8e-06" izz="1.4e-05" ixy="-3e-06" iyz="3e-06" ixz="1e-06"/>
+  </inertial>
+  <visual>
+    <origin xyz="0.006 -0.447874 0.024136" rpy="0 0 0"/>
+    <geometry>
+      <mesh filename="file://$(find robotic_description)/meshes/finger_1_2.stl" scale="0.001 0.001 0.001"/>
+    </geometry>
+    <material name="silver"/>
+  </visual>
+  <collision>
+    <origin xyz="0.006 -0.447874 0.024136" rpy="0 0 0"/>
+    <geometry>
+      <mesh filename="file://$(find robotic_description)/meshes/finger_1_2.stl" scale="0.001 0.001 0.001"/>
+    </geometry>
+  </collision>
+</link>
 <link name="WRIST_ARM_v1_1">
   <inertial>
-    <origin xyz="0.00013557693321747315 0.024520537080992555 -0.030860701686775367" rpy="0 0 0"/>
+    <origin xyz="0.00013557693321748665 0.02430753708099259 -0.030810701686775542" rpy="0 0 0"/>
     <mass value="0.4651410516079968"/>
     <inertia ixx="0.000359" iyy="0.000152" izz="0.000241" ixy="-2e-06" iyz="2.5e-05" ixz="0.0"/>
   </inertial>
   <visual>
-    <origin xyz="1.1e-05 -0.327974 -0.0259" rpy="0 0 0"/>
+    <origin xyz="1.1e-05 -0.328187 -0.02585" rpy="0 0 0"/>
     <geometry>
       <mesh filename="file://$(find robotic_description)/meshes/WRIST_ARM_v1_1.stl" scale="0.001 0.001 0.001"/>
@@ -98,5 +158,5 @@
   </visual>
   <collision>
-    <origin xyz="1.1e-05 -0.327974 -0.0259" rpy="0 0 0"/>
+    <origin xyz="1.1e-05 -0.328187 -0.02585" rpy="0 0 0"/>
     <geometry>
       <mesh filename="file://$(find robotic_description)/meshes/WRIST_ARM_v1_1.stl" scale="0.001 0.001 0.001"/>
@@ -104,65 +164,5 @@
   </collision>
 </link>
-<link name="WRIST_1">
-  <inertial>
-    <origin xyz="-6.00612610517125e-06 0.022392627588266545 -0.00018853265074284068" rpy="0 0 0"/>
-    <mass value="0.062244194694843255"/>
-    <inertia ixx="2.4e-05" iyy="2.1e-05" izz="1.8e-05" ixy="-0.0" iyz="-0.0" ixz="0.0"/>
-  </inertial>
-  <visual>
-    <origin xyz="-0.0 -0.407987 -0.0001" rpy="0 0 0"/>
-    <geometry>
-      <mesh filename="file://$(find robotic_description)/meshes/WRIST_1.stl" scale="0.001 0.001 0.001"/>
-    </geometry>
-    <material name="silver"/>
-  </visual>
-  <collision>
-    <origin xyz="-0.0 -0.407987 -0.0001" rpy="0 0 0"/>
-    <geometry>
-      <mesh filename="file://$(find robotic_description)/meshes/WRIST_1.stl" scale="0.001 0.001 0.001"/>
-    </geometry>
-  </collision>
-</link>
-<link name="finger_1_1">
-  <inertial>
-    <origin xyz="-0.0007126631883797706 0.016327909388517414 0.05456077201686823" rpy="0 0 0"/>
-    <mass value="0.0544277408008124"/>
-    <inertia ixx="1.4e-05" iyy="8e-06" izz="1.4e-05" ixy="3e-06" iyz="-3e-06" ixz="1e-06"/>
-  </inertial>
-  <visual>
-    <origin xyz="-0.006 -0.447874 0.0298" rpy="0 0 0"/>
-    <geometry>
-      <mesh filename="file://$(find robotic_description)/meshes/finger_1_1.stl" scale="0.001 0.001 0.001"/>
-    </geometry>
-    <material name="silver"/>
-  </visual>
-  <collision>
-    <origin xyz="-0.006 -0.447874 0.0298" rpy="0 0 0"/>
-    <geometry>
-      <mesh filename="file://$(find robotic_description)/meshes/finger_1_1.stl" scale="0.001 0.001 0.001"/>
-    </geometry>
-  </collision>
-</link>
-<link name="finger_1_2">
-  <inertial>
-    <origin xyz="0.0007126631883831863 0.016327909388516193 0.00023915579057530098" rpy="0 0 0"/>
-    <mass value="0.0544277408008124"/>
-    <inertia ixx="1.4e-05" iyy="8e-06" izz="1.4e-05" ixy="-3e-06" iyz="3e-06" ixz="1e-06"/>
-  </inertial>
-  <visual>
-    <origin xyz="0.006 -0.447874 0.024136" rpy="0 0 0"/>
-    <geometry>
-      <mesh filename="file://$(find robotic_description)/meshes/finger_1_2.stl" scale="0.001 0.001 0.001"/>
-    </geometry>
-    <material name="silver"/>
-  </visual>
-  <collision>
-    <origin xyz="0.006 -0.447874 0.024136" rpy="0 0 0"/>
-    <geometry>
-      <mesh filename="file://$(find robotic_description)/meshes/finger_1_2.stl" scale="0.001 0.001 0.001"/>
-    </geometry>
-  </collision>
-</link>
-<joint name="Revolute 1" type="continuous">
+<joint name="base_joint" type="continuous">
   <origin xyz="0.0 0.000487 0.0" rpy="0 0 0"/>
   <parent link="base_link"/>
@@ -170,5 +170,5 @@
   <axis xyz="0.0 -1.0 0.0"/>
 </joint>
-<joint name="Revolute 2" type="continuous">
+<joint name="shoulder_joint" type="continuous">
   <origin xyz="0.0 0.064087 0.03115" rpy="0 0 0"/>
   <parent link="SHOULDER_1"/>
@@ -176,5 +176,5 @@
   <axis xyz="0.0 -0.0 -1.0"/>
 </joint>
-<joint name="Revolute 3" type="continuous">
+<joint name="upper_lower_arm_joint" type="continuous">
   <origin xyz="-0.0 0.149904 -0.05875" rpy="0 0 0"/>
   <parent link="LOWER_ARM_1"/>
@@ -182,12 +182,6 @@
   <axis xyz="-0.0 0.0 1.0"/>
 </joint>
-<joint name="Revolute 4" type="continuous">
-  <origin xyz="-1.1e-05 0.113496 0.0535" rpy="0 0 0"/>
-  <parent link="UPPER_ARM_1"/>
-  <child link="WRIST_ARM_v1_1"/>
-  <axis xyz="-0.0 0.0 -1.0"/>
-</joint>
-<joint name="Revolute 6" type="continuous">
-  <origin xyz="1.1e-05 0.080013 -0.0258" rpy="0 0 0"/>
+<joint name="wrist joint" type="continuous">
+  <origin xyz="1.1e-05 0.0798 -0.02575" rpy="0 0 0"/>
   <parent link="WRIST_ARM_v1_1"/>
   <child link="WRIST_1"/>
@@ -208,3 +202,9 @@
   <limit upper="0.0" lower="0.0" effort="100" velocity="100"/>
 </joint>
+<joint name="upper_wrist_joint" type="continuous">
+  <origin xyz="-1.1e-05 0.113709 0.05345" rpy="0 0 0"/>
+  <parent link="UPPER_ARM_1"/>
+  <child link="WRIST_ARM_v1_1"/>
+  <axis xyz="-0.0 0.0 -1.0"/>
+</joint>
 </robot>

Commit message: Correct joint and oreintation

File: robotic_description/urdf/robotic.xacro (robot description, xacro)
@@ -11,5 +11,5 @@
   </inertial>
   <visual>
-    <origin xyz="0 0 0" rpy="0 0 0"/>
+    <origin xyz="0 0 0" rpy="1.5708 0 0"/>
     <geometry>
       <mesh filename="file://$(find robotic_description)/meshes/base_link.stl" scale="0.001 0.001 0.001"/>
@@ -18,5 +18,5 @@
   </visual>
   <collision>
-    <origin xyz="0 0 0" rpy="0 0 0"/>
+    <origin xyz="0 0 0" rpy="1.5708 0 0"/>
     <geometry>
       <mesh filename="file://$(find robotic_description)/meshes/base_link.stl" scale="0.001 0.001 0.001"/>
@@ -165,5 +165,5 @@
 </link>
 <joint name="base_joint" type="continuous">
-  <origin xyz="0.0 0.000487 0.0" rpy="0 0 0"/>
+  <origin xyz="0.0 0.000487 0.0" rpy="1.5708 0 0"/>
   <parent link="base_link"/>
   <child link="SHOULDER_1"/>
